File: Hardware/LCMXO/RAM2GS.kicad_pcb (KiCad board)
At the start: 4 copper layers, 67.3 x 48.5 mm, 64 parts, among them J1 IIgs RAM Exp., J2 JTAG, U1 LCMXO256C-3TN100C, U10 74LVC1G04GW, U11 AP2127K-1.2TRG1, U12 25F010, U2 W9812G6KH-6, U3 60M, U4 74AHCT245PW, U5 74LVC245APW, U6 74LVC245APW, U7 74LVC245APW, U8 AZ1117CH-3.3TRG1, U9 74LVC1G04GW

Commit message: Create derivative version RAM2GS
 1. Remove Garrett's Workshop trademarks from PCB front silkscreen.
 2. Add Create Common attribution PCB back silkscreen.
 3. Modify Makefile to work on Raspbian or similar Linux systems.
 4. Add README.md
Parts:
- removed the G*** at (67.2, 95.2)
Other:
- board text added: "RAM2GS Derivative by C. Kwan Orig. Design: Garrett's Workshop CC BY-SA 4.0 | github.com/svretrogames/RAM2GS"
